File: kicad/source/mt.kicad_sch (KiCad schematic)
At the start: 50 parts, among them IC1 MCP73831T-2ACI_OT, IC2 BQ29728DSER, IC3 TLV74333PDBVR, IC4 TLV9152IDR, IC5 MSPM0G3507SPMR, IC6 IS62WV1288BLL-55QLI, IC7 DAC082S085CIMMX_NOPB, IC8 SN74HC148NSR, J1 694106301002, J2 SJ1-3524N, J3 Conn_01x05_MountingPin, J4 Conn_01x09_MountingPin, Q1 CSD16406Q3, Q2 CSD16406Q3, U1 1043

Commit message: completed full schematic
Parts:
- removed J3: Conn_01x05_MountingPin, Connector_PinHeader_2.54mm:PinHeader_1x05_P2.54mm_Horizontal, symbol Connector_Generic_MountingPin:Conn_01x05_MountingPin
- removed J4: Conn_01x09_MountingPin, Connector_PinHeader_2.54mm:PinHeader_1x09_P2.54mm_Vertical, symbol Connector_Generic_MountingPin:Conn_01x09_MountingPin
- added C20, C21, C22, C23, C24, C25: 10u, Capacitor_SMD:C_0402_1005Metric, symbol Device:C
- added IC10, IC11, IC9: SN74HC148NSR, SN74HC148NSR:SOIC127P780X200-16N, symbol SN74HC148NSR:SN74HC148NSR
- added J3: Conn_01x05_Pin, Connector_PinHeader_2.54mm:PinHeader_1x05_P2.54mm_Horizontal, symbol Connector:Conn_01x05_Pin
- added J4: Conn_01x09_Pin, Connector_PinSocket_2.54mm:PinSocket_1x09_P2.54mm_Vertical, symbol Connector:Conn_01x09_Pin
- added R17, R18, R19, R20, R21, R22, R23, R24, R25, R26, R27, R28, R29, R30, R31, R32, R33, R34, R35, R36, R37, R38, R39, R40, R41, R42, R43, R44, R45, R46, R47, R48, R49, R5, R6: 100k, Resistor_SMD:R_0402_1005Metric, symbol Device:R_US
- added S10, S11, S12, S13, S14, S15, S16, S17, S18, S19, S20, S21, S22, S23, S24, S25, S26, S27, S28, S29, S3, S30, S31, S32, S33, S34, S35, S4, S5, S6, S7, S8, S9: TL6800AF160QJ, TL6800AF160QJ:TL6800AF160QJ, symbol TL6800AF160QJ:TL6800AF160QJ
- renumbered R8 to R10, R9 to R11, R10 to R12, R11 to R13, R12 to R14, R13 to R15, R14 to R16, R5 to R7, R6 to R8, R7 to R9
Connections:
- net GND: now also IC6.22 (~{CS1}), IC6.24 (~{OE}), IC7.6 (GND), IC8.5 (EI), IC8.8 (GND), C20.2, C21.2, C22.2, C23.2, C24.2, C25.2, IC10.5 (EI), IC10.8 (GND), IC11.5 (EI), IC11.8 (GND), IC9.5 (EI), IC9.8 (GND), J3.1 (Pin_1), J4.3 (Pin_3), R6.2, S10.3, S10.4, S11.3, S11.4, S12.3, S12.4, S13.3, S13.4, S14.3, S14.4, S15.3, S15.4, S16.3, S16.4, S17.3, S17.4, S18.3, S18.4, S19.3, S19.4, S20.3, S20.4, S21.3, S21.4, S22.3, S22.4, S23.3, S23.4, S24.3, S24.4, S25.3, S25.4, S26.3, S26.4, S27.3, S27.4, S28.3, S28.4, S29.3, S29.4, S3.3, S3.4, S30.3, S30.4, S31.3, S31.4, S32.3, S32.4, S33.3, S33.4, S34.3, S34.4, S35.3, S35.4, S4.3, S4.4, S5.3, S5.4, S6.3, S6.4, S7.3, S7.4, S8.3, S8.4, S9.3, S9.4
- net NRST: now also J3.3 (Pin_3)
- net SWCLK: now also J3.5 (Pin_5)
- net SWDIO: now also J3.4 (Pin_4)
- net VBAT: now also IC5.17 (PA21_/_A1_7_/_VREF-), R5.1, R6.1; no longer C4.1, IC3.1 (IN), IC3.3 (EN), S1.2
- net VDD: now also C15.1, C16.1, C18.1, C19.1, IC5.40 (VDD), IC6.32 (VDD), IC7.1 (VA), IC7.7 (VREFIN), IC8.16 (VCC), C20.1, C21.1, C22.1, C23.1, C24.1, C25.1, IC10.16 (VCC), IC11.16 (VCC), IC9.16 (VCC), J3.2 (Pin_2), J4.1 (Pin_1), R17.1, R18.1, R19.1, R20.1, R21.1, R22.1, R23.1, R24.1, R25.1, R26.1, R27.1, R28.1, R29.1, R30.1, R31.1, R32.1, R33.1, R34.1, R35.1, R36.1, R37.1, R38.1, R39.1, R40.1, R41.1, R42.1, R43.1, R44.1, R45.1, R46.1, R47.1, R48.1, R49.1
- net SPI1_SCK: now reaches IC7.10 (SCLK)
- net SPI1_SCK: now also IC5.10 (PA17_/_A1_2)
- net SPI1_PICO: now reaches IC7.8 (DIN)
- net SPI1_PICO: now also IC5.11 (PA18_/_A1_3)
- net ~SYNC: now reaches IC7.9 (~{SYNC})
- net ~SYNC: now also IC5.9 (PA16_/A1_1_/FCC_IN)
- net SPI0_PICO: now reaches IC5.14 (PB17_/_A1_4)
- net SPI0_PICO: now also J4.5 (Pin_5)
- net SPI0_SCK: now reaches IC5.15 (PB18_/_A1_5)
- net SPI0_SCK: now also J4.4 (Pin_4)
- net E0_GS: now reaches IC5.19 (PB20_/_A0_6)
- net E0_GS: now also IC8.14 (GS)
- net E1_GS: now reaches IC5.20 (PB21)
- net E1_GS: now also IC9.14 (GS)
- net E2_GS: now reaches IC5.21 (PB22)
- net E2_GS: now also IC10.14 (GS)
- net E3_GS: now reaches IC5.22 (PB23)
- net E3_GS: now also IC11.14 (GS)
- net E2_0: now reaches IC5.25 (PA24_/_A0_3)
- net E2_0: now also IC10.9 (A0)
- net E2_1: now reaches IC5.26 (PA25_/_A0_2)
- net E2_1: now also IC10.7 (A1)
- net SPI0_CS0: now reaches IC5.27 (PB25_/_A0_4)
- net SPI0_CS0: now also J4.6 (Pin_6)
- net E2_2: now reaches IC5.30 (PA26_/_A0_1)
- net E2_2: now also IC10.6 (A2)
- net E3_0: now reaches IC5.31 (PA27/_A0_0)
- net E3_0: now also IC11.9 (A0)
- net E0_0: now reaches IC5.33 (PA0_/_FCC_IN)
- net E0_0: now also IC8.9 (A0)
- net E0_1: now reaches IC5.34 (PA1)
- net E0_1: now also IC8.7 (A1)
- net E3_1: now reaches IC5.35 (PA28)
- net E3_1: now also IC11.7 (A1)
- net E3_2: now reaches IC5.36 (PA29)
- net E3_2: now also IC11.6 (A2)
- net Ex_0: now reaches IC5.37 (PA30)
- net Ex_0: now also R48.2, S34.1, S34.2
- net Ex_1: now reaches IC5.39 (PA31_/_CLK_OUT)
- net Ex_1: now also R49.2, S35.1, S35.2
- net E0_2: now reaches IC5.42 (PA2_/_ROSC)
- net E0_2: now also IC8.6 (A2)
- net E1_0: now reaches IC5.43 (PA3_/_LFXIN)
- net E1_0: now also IC9.9 (A0)
- net E1_1: now reaches IC5.44 (PA4_/_LFCLK_IN_/_LFXOUT)
- net E1_1: now also IC9.7 (A1)
- net E1_2: now reaches IC5.45 (PA5_/_HFXIN_/_FCC_IN)
- net E1_2: now also IC9.6 (A2)
- net RAM_WR: now reaches IC5.46 (PA6_/_HFCLK_IN_/_HFXOUT)
- net RAM_WR: now also IC6.29 (~{WE})
- net RAM_EN: now reaches IC5.49 (PA7_/_CLK_OUT)
- net RAM_EN: now also IC6.30 (CS2)
- net I/O4: now reaches IC5.5 (PA12_/_FCC_IN)
- net I/O4: now also IC6.18 (I/O4)
- net I/O0: now reaches IC5.54 (PA8)
- net I/O0: now also IC6.13 (I/O0)
- net I/O1: now reaches IC5.55 (PA9_/_RTC_OUT_/_CLK_OUT)
- net I/O1: now also IC6.14 (I/O1)
- net I/O2: now reaches IC5.56 (PA10_/_CLK_OUT)
- net I/O2: now also IC6.15 (I/O2)
- net I/O3: now reaches IC5.57 (PA11)
- net I/O3: now also IC6.17 (I/O3)
- net I/O5: now reaches IC5.6 (PA13)
- net I/O5: now also IC6.19 (I/O5)
- net I/O6: now reaches IC5.7 (PA14_/_CLK_OUT_/_A0_12)
- net I/O6: now also IC6.20 (I/O6)
- net I/O7: now reaches IC5.8 (PA15_/_A1_0)
- net I/O7: now also IC6.21 (I/O7)
- net at R16.2, S2.1, S2.2: now also IC8.10 (0)
- net at IC8.1 (4): now also R17.2, S3.1, S3.2
- net at IC8.11 (1): now also R18.2, S4.1, S4.2
- net at IC8.12 (2): now also R20.2, S6.1, S6.2
- net at IC8.13 (3): now also R22.2, S8.1, S8.2
- net at IC8.2 (5): now also R19.2, S5.1, S5.2
- net at IC8.3 (6): now also R21.2, S7.1, S7.2
- net at IC8.4 (7): now also R23.2, S9.1, S9.2
- new net: C4.1, IC3.1 (IN), IC3.3 (EN), R5.2, S1.2
- new net: IC11.1 (4), R41.2, S27.1, S27.2
- new net: IC9.1 (4), R25.2, S11.1, S11.2
- new net: IC9.10 (0), R24.2, S10.1, S10.2
- new net: IC9.11 (1), R26.2, S12.1, S12.2
- new net: IC9.12 (2), R28.2, S14.1, S14.2
- new net: IC9.13 (3), R30.2, S16.1, S16.2
- new net: IC9.2 (5), R27.2, S13.1, S13.2
- new net: IC9.3 (6), R29.2, S15.1, S15.2
- new net: IC9.4 (7), R31.2, S17.1, S17.2
- new net: IC10.1 (4), R33.2, S19.1, S19.2
- new net: IC10.2 (5), R35.2, S21.1, S21.2
- new net: IC11.12 (2), R44.2, S30.1, S30.2
- new net: IC11.13 (3), R46.2, S32.1, S32.2
- new net: IC10.11 (1), R34.2, S20.1, S20.2
- new net: IC10.3 (6), R37.2, S23.1, S23.2
- new net: IC11.3 (6), R45.2, S31.1, S31.2
- new net: IC10.12 (2), R36.2, S22.1, S22.2
- new net: IC10.4 (7), R39.2, S25.1, S25.2
- new net: IC11.2 (5), R43.2, S29.1, S29.2
- new net: IC10.13 (3), R38.2, S24.1, S24.2
- new net: IC11.10 (0), R40.2, S26.1, S26.2
- new net: IC11.4 (7), R47.2, S33.1, S33.2
- new net: IC11.11 (1), R42.2, S28.1, S28.2
- new net: IC10.10 (0), R32.2, S18.1, S18.2
- no-connect marks 18 -> 30
Other:
- note added: "Buttons"
- note added: "Digital"
- note added: "Microcontroller"
- note added: "Rank 0"
- note added: "Rank 1"
- note added: "Rank 2"
- note added: "Rank 3"
- note added: "SRAM"
- note added: "Serial Peripherals"
- note removed: "Remember to add JLCPCB part #s to all SMD parts!"
- moved on the sheet: C1, C10, C11, C12, C13, C14, C15, C16, C17, C18, C19, C2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
